File: Project/FPGAAudio/FPGAAudio.kicad_sch (KiCad schematic)
At the start: 24 parts, among them J1 Conn_01x02_Pin, J2 Conn_01x08_Pin, SW1 SW_SPDT, SW2 SW_SPDT, U1 PAM8403D

Commit message: ye
Parts:
- added C10, C11, C12, C9: 220pF, symbol Device:C_Small
- added C13: 0.1u, symbol Device:C_Small
- added C14: 1u, symbol Device:C_Small
- added FB1, FB2, FB3, FB4: FerriteBead_Small, symbol Device:FerriteBead_Small
- added R8: 47, symbol Device:R_Small
- C4: value 0.1u -> 1u
- R2, R3: value 100k -> 33k
Connections:
- net GND: now also C10.2, C11.2, C12.1, C13.1, C14.1, C9.1
- net LOUT+: now also C9.2, FB1.2; no longer U1.1 (LOUT+)
- net LOUT-: now also C10.1, FB2.2; no longer U1.3 (LOUT-)
- net ROUT+: now also C11.1, FB4.2; no longer U1.16 (ROUT+)
- net ROUT-: now also C12.2, FB3.2; no longer U1.14 (ROUT-)
- net VCC33: now also C13.2, R8.1; no longer J2.7 (Pin_7), R6.1, R7.1
- net VCC50: now also R6.1, R7.1; no longer U1.4 (PVDD)
- new net: J2.7 (Pin_7), R8.2
- new net: FB1.1, U1.1 (LOUT+)
- new net: FB3.1, U1.14 (ROUT-)
- new net: FB4.1, U1.16 (ROUT+)
- new net: FB2.1, U1.3 (LOUT-)
- new net: C14.2, U1.4 (PVDD)
Other:
- note added: "Todo : LM386 based headphone amplifier with 6 input double pole switch Debouncing capacitors for all buttons verification"
- moved on the sheet: C1, C2, C3, C4, C5, C6, C7, C8, LS1, LS2, R1, R2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

Commit message: yeyeeye
Parts:
- added C15, C17: 0.1u, symbol Device:C_Small
- added C16: 100u, symbol Device:C_Small
- added C18: 10u, symbol Device:C_Small
- added C19: 0.047u, symbol Device:C_Small
- added C21: 470u, symbol Device:C_Polarized
- added J3: AudioJack3_Ground_Switch, symbol Connector_Audio:AudioJack3_Ground_Switch
- added R10, R11: 100k, symbol Device:R_Small
- added R9: 10, symbol Device:R_Small
- added SW3: SW_SPDT, symbol Switch:SW_SPDT
- added U2: LM386, symbol Amplifier_Audio:LM386
Connections:
- net GND: now also C16.1, C17.1, C18.2, J3.G, J3.S, R10.1, R11.2, R9.2, U2.2 (-), U2.4 (GND)
- net VCC50: now also C16.2, C17.2, U2.6 (V+)
- net SpeakerIN: now reaches C2.1, C3.1
- net SpeakerIN: now also R10.2, SW3.1 (A); no longer RV1.2
- new net: C15.2, U2.3 (+)
- new net: C19.2, C21.1, U2.5
- new net: C18.1, U2.7 (BYPASS)
- new net: C19.1, R9.1
- new net HOut: C21.2, J3.R, J3.T
- new net HeadphoneIN: C15.1, R11.1, SW3.3 (C)
- new net RCout: RV1.2, SW3.2 (B)
- no-connect marks 1 -> 6
Other:
- note added: "(Headphone)"
- note added: "(Speaker)"
- note added: "Analog Stage"
- note added: "Class AB"
- note added: "Class D"
- note added: "RC"
- note added: "Switch"
- note removed: "Audio Stage"
- note removed: "ERC"
- note removed: "Todo : LM386 based headphone amplifier with 6 input double pole switch Debouncing capacitors for all buttons verification"
- moved on the sheet: C1, C10, C11, C12, C13, C14, C2, C3, C4, C5, C6, C7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
